File: letter-k.sch (KiCad schematic (older format))
At the start: 28 parts

Commit message: Connect rest of pins on the buffer to VCC/Gnd. Resize copper plane to cover more of the Pico after its move. Fix a couple of unconnected tracks. PCB version on silkscreen to v0.2.
Also updates schematic with capacitor footprint changes.
Parts:
- C1, C10, C11, C12, C13, C14, C2, C3, C4, C5, C6, C7, C8, C9: footprint Capacitor_THT:CP_Radial_D4.0mm_P2.00mm -> Capacitor_THT:C_Disc_D4.7mm_W2.5mm_P5.00mm
Changed lines of the file:
@@
 F 0 "C1" H 2618 1346 50  0000 L CNN
 F 1 "0.1uF" H 2618 1255 50  0000 L CNN
-F 2 "Capacitor_THT:CP_Radial_D4.0mm_P2.00mm" H 2538 1150 50  0001 C CNN
+F 2 "Capacitor_THT:C_Disc_D4.7mm_W2.5mm_P5.00mm" H 2538 1150 50  0001 C CNN
 F 3 "~" H 2500 1300 50  0001 C CNN
 	1    2500 1300
@@
 F 0 "C2" H 2618 2146 50  0000 L CNN
 F 1 "0.1uF" H 2618 2055 50  0000 L CNN
-F 2 "Capacitor_THT:CP_Radial_D4.0mm_P2.00mm" H 2538 1950 50  0001 C CNN
+F 2 "Capacitor_THT:C_Disc_D4.7mm_W2.5mm_P5.00mm" H 2538 1950 50  0001 C CNN
 F 3 "~" H 2500 2100 50  0001 C CNN
 	1    2500 2100
@@
 F 0 "C3" H 2618 2946 50  0000 L CNN
 F 1 "0.1uF" H 2618 2855 50  0000 L CNN
-F 2 "Capacitor_THT:CP_Radial_D4.0mm_P2.00mm" H 2538 2750 50  0001 C CNN
+F 2 "Capacitor_THT:C_Disc_D4.7mm_W2.5mm_P5.00mm" H 2538 2750 50  0001 C CNN
 F 3 "~" H 2500 2900 50  0001 C CNN
 	1    2500 2900
@@
 F 0 "C4" H 2618 3746 50  0000 L CNN
 F 1 "0.1uF" H 2618 3655 50  0000 L CNN
-F 2 "Capacitor_THT:CP_Radial_D4.0mm_P2.00mm" H 2538 3550 50  0001 C CNN
+F 2 "Capacitor_THT:C_Disc_D4.7mm_W2.5mm_P5.00mm" H 2538 3550 50  0001 C CNN
 F 3 "~" H 2500 3700 50  0001 C CNN
 	1    2500 3700
@@
 F 0 "C5" H 2618 4546 50  0000 L CNN
 F 1 "0.1uF" H 2618 4455 50  0000 L CNN
-F 2 "Capacitor_THT:CP_Radial_D4.0mm_P2.00mm" H 2538 4350 50  0001 C CNN
+F 2 "Capacitor_THT:C_Disc_D4.7mm_W2.5mm_P5.00mm" H 2538 4350 50  0001 C CNN
 F 3 "~" H 2500 4500 50  0001 C CNN
 	1    2500 4500
@@
 F 0 "C6" H 2618 5346 50  0000 L CNN
 F 1 "0.1uF" H 2618 5255 50  0000 L CNN
-F 2 "Capacitor_THT:CP_Radial_D4.0mm_P2.00mm" H 2538 5150 50  0001 C CNN
+F 2 "Capacitor_THT:C_Disc_D4.7mm_W2.5mm_P5.00mm" H 2538 5150 50  0001 C CNN
 F 3 "~" H 2500 5300 50  0001 C CNN
 	1    2500 5300
@@
 F 0 "C7" H 2618 6146 50  0000 L CNN
 F 1 "0.1uF" H 2618 6055 50  0000 L CNN
-F 2 "Capacitor_THT:CP_Radial_D4.0mm_P2.00mm" H 2538 5950 50  0001 C CNN
+F 2 "Capacitor_THT:C_Disc_D4.7mm_W2.5mm_P5.00mm" H 2538 5950 50  0001 C CNN
 F 3 "~" H 2500 6100 50  0001 C CNN
 	1    2500 6100
@@
 F 0 "C8" H 4618 3746 50  0000 L CNN
 F 1 "0.1uF" H 4618 3655 50  0000 L CNN
-F 2 "Capacitor_THT:CP_Radial_D4.0mm_P2.00mm" H 4538 3550 50  0001 C CNN
+F 2 "Capacitor_THT:C_Disc_D4.7mm_W2.5mm_P5.00mm" H 4538 3550 50  0001 C CNN
 F 3 "~" H 4500 3700 50  0001 C CNN
 	1    4500 3700
@@
 F 0 "C9" H 5968 2946 50  0000 L CNN
 F 1 "0.1uF" H 5968 2855 50  0000 L CNN
-F 2 "Capacitor_THT:CP_Radial_D4.0mm_P2.00mm" H 5888 2750 50  0001 C CNN
+F 2 "Capacitor_THT:C_Disc_D4.7mm_W2.5mm_P5.00mm" H 5888 2750 50  0001 C CNN
 F 3 "~" H 5850 2900 50  0001 C CNN
 	1    5850 2900
@@
 F 0 "C10" H 5968 4546 50  0000 L CNN
 F 1 "0.1uF" H 5968 4455 50  0000 L CNN
-F 2 "Capacitor_THT:CP_Radial_D4.0mm_P2.00mm" H 5888 4350 50  0001 C CNN
+F 2 "Capacitor_THT:C_Disc_D4.7mm_W2.5mm_P5.00mm" H 5888 4350 50  0001 C CNN
 F 3 "~" H 5850 4500 50  0001 C CNN
 	1    5850 4500
@@
 F 0 "C11" H 7318 2146 50  0000 L CNN
 F 1 "0.1uF" H 7318 2055 50  0000 L CNN
-F 2 "Capacitor_THT:CP_Radial_D4.0mm_P2.00mm" H 7238 1950 50  0001 C CNN
+F 2 "Capacitor_THT:C_Disc_D4.7mm_W2.5mm_P5.00mm" H 7238 1950 50  0001 C CNN
 F 3 "~" H 7200 2100 50  0001 C CNN
 	1    7200 2100
@@
 F 0 "C12" H 7318 5346 50  0000 L CNN
 F 1 "0.1uF" H 7318 5255 50  0000 L CNN
-F 2 "Capacitor_THT:CP_Radial_D4.0mm_P2.00mm" H 7238 5150 50  0001 C CNN
+F 2 "Capacitor_THT:C_Disc_D4.7mm_W2.5mm_P5.00mm" H 7238 5150 50  0001 C CNN
 F 3 "~" H 7200 5300 50  0001 C CNN
 	1    7200 5300
@@
 F 0 "C13" H 8668 1346 50  0000 L CNN
 F 1 "0.1uF" H 8668 1255 50  0000 L CNN
-F 2 "Capacitor_THT:CP_Radial_D4.0mm_P2.00mm" H 8588 1150 50  0001 C CNN
+F 2 "Capacitor_THT:C_Disc_D4.7mm_W2.5mm_P5.00mm" H 8588 1150 50  0001 C CNN
 F 3 "~" H 8550 1300 50  0001 C CNN
 	1    8550 1300
@@
 F 0 "C14" H 8668 6146 50  0000 L CNN
 F 1 "0.1uF" H 8668 6055 50  0000 L CNN
-F 2 "Capacitor_THT:CP_Radial_D4.0mm_P2.00mm" H 8588 5950 50  0001 C CNN
+F 2 "Capacitor_THT:C_Disc_D4.7mm_W2.5mm_P5.00mm" H 8588 5950 50  0001 C CNN
 F 3 "~" H 8550 6100 50  0001 C CNN
 	1    8550 6100
