File: namebadge.kicad_pcb (KiCad board)
At the start: 2 copper layers, 73.7 x 132.1 mm, 35 parts, among them IC1 SN74AHCT125N, J1 Barrel_Jack, SW1 SW_Push, U1 Pico

Commit message: Ground /OE on level shifter.
Fixes #1.
Connections:
- IC1 pad 1: Net-(IC1-Pad1) -> GND
