File: namebadge.sch (KiCad schematic (older format))
At the start: 7 parts, among them IC1 SN74AHCT125N, J1 Barrel_Jack, SW1 SW_Push, U1 Pico

Commit message: fix dropped connection to gpio
Connections:
- net GND: no longer IC1.12 (4A), U1.1 (GPIO0)
- new net: IC1.12 (4A), U1.1 (GPIO0)
Changed lines of the file:
@@
 Wire Wire Line
 	3250 1850 3250 2350
-Wire Wire Line
-	2800 1650 4000 1650
-Wire Wire Line
-	4000 1650 4000 1550
 $Comp
 L power:VCC #PWR0101
 U 1 1 6053EF5E
-P 4000 1550
-F 0 "#PWR0101" H 4000 1400 50  0001 C CNN
-F 1 "VCC" H 4015 1723 50  0000 C CNN
-F 2 "" H 4000 1550 50  0001 C CNN
-F 3 "" H 4000 1550 50  0001 C CNN
-	1    4000 1550
+P 2950 900
+F 0 "#PWR0101" H 2950 750 50  0001 C CNN
+F 1 "VCC" H 2965 1073 50  0000 C CNN
+F 2 "" H 2950 900 50  0001 C CNN
+F 3 "" H 2950 900 50  0001 C CNN
+	1    2950 900
 	1    0    0    -1
 $EndComp
@@
 	1400 1850 1050 1850
 Wire Wire Line
-	1050 1850 1050 1250
-Wire Wire Line
 	1050 1850 1050 2350
 Wire Wire Line
 	1050 2350 1400 2350
-Connection ~ 1050 1850
 Wire Wire Line
 	1050 2350 1050 2850
@@
 L power:GND #PWR0103
 U 1 1 60540BCC
-P 1050 1100
-F 0 "#PWR0103" H 1050 850 50  0001 C CNN
-F 1 "GND" H 1055 927 50  0000 C CNN
-F 2 "" H 1050 1100 50  0001 C CNN
-F 3 "" H 1050 1100 50  0001 C CNN
-	1    1050 1100
-	-1   0    0    1
+P 1050 3600
+F 0 "#PWR0103" H 1050 3350 50  0001 C CNN
+F 1 "GND" H 1055 3427 50  0000 C CNN
+F 2 "" H 1050 3600 50  0001 C CNN
+F 3 "" H 1050 3600 50  0001 C CNN
+	1    1050 3600
+	1    0    0    -1
 $EndComp
 NoConn ~ 2800 1950
@@
 L power:GND #PWR01
 U 1 1 6073F12A
-P 4200 3450
-F 0 "#PWR01" H 4200 3200 50  0001 C CNN
-F 1 "GND" H 4205 3277 50  0000 C CNN
-F 2 "" H 4200 3450 50  0001 C CNN
-F 3 "" H 4200 3450 50  0001 C CNN
-	1    4200 3450
+P 4850 3450
+F 0 "#PWR01" H 4850 3200 50  0001 C CNN
+F 1 "GND" H 4855 3277 50  0000 C CNN
+F 2 "" H 4850 3450 50  0001 C CNN
+F 3 "" H 4850 3450 50  0001 C CNN
+	1    4850 3450
 	1    0    0    -1
 $EndComp
@@
 Wire Wire Line
 	1400 1650 1200 1650
-Wire Wire Line
-	1200 1650 1200 1250
 $Comp
 L Device:CP C15
@@
 	-1   0    0    1
 $EndComp
-Wire Wire Line
-	1200 1250 3250 1250
 NoConn ~ 2800 3550
 $Comp
@@
 	5550 2550 5550 3300
 Wire Wire Line
-	4200 3300 5550 3300
-Connection ~ 4200 3300
-Wire Wire Line
-	4200 3300 4200 3450
-Wire Wire Line
 	3850 3050 3900 3050
 Wire Wire Line
@@
 	6300 3550 6050 3550
 Wire Wire Line
-	1200 3550 1200 4250
-Wire Wire Line
-	1200 4250 1300 4250
-Wire Wire Line
-	1200 3550 1400 3550
+	1250 3550 1250 4250
+Wire Wire Line
+	1250 4250 1300 4250
+Wire Wire Line
+	1250 3550 1400 3550
 $Comp
 L power:GND #PWR0120
@@
 NoConn ~ 2800 1750
 Wire Wire Line
-	4000 1650 4800 1650
-Wire Wire Line
-	4800 1650 4800 2050
-Connection ~ 4000 1650
+	4800 900  4800 2050
 Connection ~ 4800 2050
 Wire Wire Line
 	4800 2050 5400 2050
 Wire Wire Line
-	1200 1250 1050 1250
-Connection ~ 1200 1250
-Connection ~ 1050 1250
-Wire Wire Line
-	1050 1250 1050 1100
-Wire Wire Line
-	5850 1500 5850 1850
+	5850 900  5850 1850
 $Comp
 L power:VCC #PWR0119
 U 1 1 6068FE64
-P 5850 1500
-F 0 "#PWR0119" H 5850 1350 50  0001 C CNN
-F 1 "VCC" H 5865 1673 50  0000 C CNN
-F 2 "" H 5850 1500 50  0001 C CNN
-F 3 "" H 5850 1500 50  0001 C CNN
-	1    5850 1500
-	1    0    0    -1
-$EndComp
-Wire Wire Line
-	3250 1850 3250 1250
-Connection ~ 3250 1850
-Connection ~ 3250 1250
-Wire Wire Line
-	3250 1250 5700 1250
+P 5850 900
+F 0 "#PWR0119" H 5850 750 50  0001 C CNN
+F 1 "VCC" H 5865 1073 50  0000 C CNN
+F 2 "" H 5850 900 50  0001 C CNN
+F 3 "" H 5850 900 50  0001 C CNN
+	1    5850 900
+	1    0    0    -1
+$EndComp
+Wire Wire Line
+	1050 3600 1050 3350
+Wire Wire Line
+	1200 1650 1200 1250
+Wire Wire Line
+	1200 1250 5700 1250
+Connection ~ 1050 3350
+$Comp
+L power:GND #PWR?
+U 1 1 607F0923
+P 3250 3600
+F 0 "#PWR?" H 3250 3350 50  0001 C CNN
+F 1 "GND" H 3255 3427 50  0000 C CNN
+F 2 "" H 3250 3600 50  0001 C CNN
+F 3 "" H 3250 3600 50  0001 C CNN
+	1    3250 3600
+	1    0    0    -1
+$EndComp
+Wire Wire Line
+	3250 3600 3250 3350
+Connection ~ 3250 3350
+Wire Wire Line
+	2950 900  2950 1650
+Wire Wire Line
+	2950 1650 2800 1650
+$Comp
+L power:VCC #PWR?
+U 1 1 607F7552
+P 4800 900
+F 0 "#PWR?" H 4800 750 50  0001 C CNN
+F 1 "VCC" H 4815 1073 50  0000 C CNN
+F 2 "" H 4800 900 50  0001 C CNN
+F 3 "" H 4800 900 50  0001 C CNN
+	1    4800 900
+	1    0    0    -1
+$EndComp
+Wire Wire Line
+	4200 3300 4850 3300
+Connection ~ 4850 3300
+Wire Wire Line
+	4850 3300 5550 3300
+Wire Wire Line
+	4850 3300 4850 3450
 $EndSCHEMATC

Commit message: Ground /OE on level shifter.
Fixes #1.
Parts:
- IC1: symbol Mouser:SN74AHCT125N -> SamacSys_Parts:SN74AHCT125N
Connections:
- net GND: now also IC1.1 (1~OE)
- no-connect marks 41 -> 40
Changed lines of the file:
@@
 	5850 2300 6300 2300
 $Comp
-L Mouser:SN74AHCT125N IC1
+L SamacSys_Parts:SN74AHCT125N IC1
 U 1 1 60732053
 P 4300 2450
@@
 NoConn ~ 4300 2650
 NoConn ~ 4300 2550
-NoConn ~ 4300 2450
 $Comp
 L Connector:Barrel_Jack J1
@@
 Wire Wire Line
 	4850 3300 4850 3450
+Wire Wire Line
+	4200 2450 4300 2450
+Wire Wire Line
+	4200 3050 4200 2450
 $EndSCHEMATC
